File: RocketTracker.kicad_pcb (KiCad board)
At the start: 2 copper layers, 58.9 x 79.8 mm, 38 parts, among them J1 HW_SERIAL, J10 ANT, J2 GPS_SERIAL, J3 LAUNCH1, J4 LAUNCH2, J5 I2C_PRESSURE, J6 Micro_SD_Card, J7 PWR_IN, J8 I2C_GYRO, J9 I2C_RTC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

Commit message: Edited the PCB design
Parts:
- moved SW2 25.2 mm to (143.8, 62.0)
- moved J6 22.7 mm to (146.1, 83.6)
- moved C6 21.7 mm to (145.0, 70.4), turned to 270 degrees
- moved R6 18.3 mm to (120.1, 108.7)
- moved R1 17.1 mm to (137.2, 69.3), turned to 180 degrees
- moved J1 16.1 mm to (151.6, 69.3)
- moved SW1 15.8 mm to (136.1, 62.0)
- moved Q4 14.6 mm to (122.2, 113.3), turned to 270 degrees
- moved R3 13.5 mm to (134.6, 108.7)
- moved R4 11.8 mm to (137.7, 118.9), turned to 180 degrees
- moved D1 11.0 mm to (142.7, 113.3), turned to 270 degrees
- moved C3 10.9 mm to (142.7, 102.9), turned to 90 degrees
- moved J10 10.9 mm to (150.9, 92.7)
- moved R7 10.5 mm to (123.2, 118.9), turned to 180 degrees
- moved Q2 10.2 mm to (136.7, 113.3), turned to 270 degrees
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Connections:
- J6 pad 1: (no net) -> Net-(J6-Pad1)
- J6 pad 8: (no net) -> Net-(J6-Pad8)
- U1 pad 10: (no net) -> Net-(U1-Pad10)
- U1 pad 11: (no net) -> Net-(U1-Pad11)
- U1 pad 17: (no net) -> Net-(U1-Pad17)
- U1 pad 18: (no net) -> Net-(U1-Pad18)
- U1 pad 19: (no net) -> Net-(U1-Pad19)
- U1 pad 20: (no net) -> Net-(U1-Pad20)
- U1 pad 21: (no net) -> Net-(U1-Pad21)
- U1 pad 22: (no net) -> Net-(U1-Pad22)
- U1 pad 23: (no net) -> Net-(U1-Pad23)
- U1 pad 24: (no net) -> Net-(U1-Pad24)
- U1 pad 26: (no net) -> Net-(U1-Pad26)
- U1 pad 32: (no net) -> Net-(U1-Pad32)
- U1 pad 33: (no net) -> Net-(U1-Pad33)
- U1 pad 36: (no net) -> Net-(U1-Pad36)
- U1 pad 4: (no net) -> Net-(U1-Pad4)
- U1 pad 5: (no net) -> Net-(U1-Pad5)
- U1 pad 9: (no net) -> Net-(U1-Pad9)
- U2 pad 11: (no net) -> Net-(U2-Pad11)
- U2 pad 12: (no net) -> Net-(U2-Pad12)
- U2 pad 15: (no net) -> Net-(U2-Pad15)
- U2 pad 16: (no net) -> Net-(U2-Pad16)
- U2 pad 7: (no net) -> Net-(U2-Pad7)
Routing:
- net GND: track 132.6 -> 0.58 mm, vias 22 -> 0
- net +3V3: track 316.6 -> 229.5 mm, vias 8 -> 12
- net Net-(Q4-Pad3): track 44.4 -> 7.10 mm, vias 2 -> 0
- net Net-(Q2-Pad3): track 29.7 -> 7.10 mm, vias 2 -> 0
- net Net-(SW2-Pad2): track 18.6 -> 37.1 mm, vias 0 -> 1
- net CS0: track 44.7 -> 26.3 mm
- net LORA_RESET: track 32.4 -> 19.8 mm
- net Net-(R1-Pad2): track 50.2 -> 39.6 mm, vias 2 -> 3
- net CS1: track 25.5 -> 17.0 mm, vias 0 -> 2
- net MOSI: track 68.0 -> 75.7 mm, vias 4 -> 5
- net Net-(J10-Pad1): track 26.4 -> 34.1 mm
- net +BATT: track 66.6 -> 58.9 mm, vias 0 -> 2
- net MISO: track 60.9 -> 68.2 mm, vias 2 -> 4
- net HW_TX: track 32.9 -> 28.2 mm
- net GPSTX: track 59.0 -> 63.2 mm, vias 2 -> 1
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- added copper zone on B.Cu, net GND
Other:
- board size 58.9 x 79.8 mm -> 58.9 x 74.2 mm
- rule trace_min: 0.2 -> 0.25
- board text added: "+"
- board text added: "-"
- board text added: "CONNECT ANTENNA BEFORE TX!"
- board text added: "HARWELL ROCKET CLUB TRACKER V2"
- board text added: "SCL"
- board text added: "SDA"
- board text added: "Will Furnell + Ryan Smith 2020"
