File: RocketTracker.sch (KiCad schematic (older format))
At the start: 36 parts, among them J1 HW_SERIAL, J10 ANT, J2 GPS_SERIAL, J3 LAUNCH1, J4 LAUNCH2, J5 I2C_PRESSURE, J6 SD_Card, J7 PWR_IN, J8 I2C_GYRO, J9 I2C_RTC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

Commit message: Update PCB
Parts:
- J3, J4: footprint Connector_PinSocket_2.54mm:PinSocket_1x02_P2.54mm_Vertical -> Connector_Wire:SolderWirePad_1x02_P3.81mm_Drill1mm
- J5, J8, J9: footprint Connector_PinSocket_2.54mm:PinSocket_1x04_P2.54mm_Vertical -> custom:PinSocket_1x04_P2.54mm_Vertical
- J7: footprint Connector:Banana_Jack_2Pin -> Connector_Wire:SolderWirePad_1x02_P3.81mm_Drill1mm
- SW1, SW2: footprint (none) -> button:FSM4JRT
- U3: footprint RF_Module:HOPERF_RFM69HW -> lm1117t-3.3_nopb:TO254P470X1028X1955-3P
Connections:
- net GND: now also J4.2 (Pin_2); no longer J4.1 (Pin_1)
- net LAUNCH2_OUT: now also J4.1 (Pin_1); no longer J4.2 (Pin_2)
Changed lines of the file:
@@
 F 0 "J3" H 10328 3876 50  0000 L CNN
 F 1 "LAUNCH1" H 10328 3785 50  0000 L CNN
-F 2 "Connector_PinSocket_2.54mm:PinSocket_1x02_P2.54mm_Vertical" H 10300 3900 50  0001 C CNN
+F 2 "Connector_Wire:SolderWirePad_1x02_P3.81mm_Drill1mm" H 10300 3900 50  0001 C CNN
 F 3 "~" H 10300 3900 50  0001 C CNN
 	1    10300 3900
@@
 F 0 "J4" H 10328 4226 50  0000 L CNN
 F 1 "LAUNCH2" H 10328 4135 50  0000 L CNN
-F 2 "Connector_PinSocket_2.54mm:PinSocket_1x02_P2.54mm_Vertical" H 10300 4250 50  0001 C CNN
+F 2 "Connector_Wire:SolderWirePad_1x02_P3.81mm_Drill1mm" H 10300 4250 50  0001 C CNN
 F 3 "~" H 10300 4250 50  0001 C CNN
 	1    10300 4250
@@
 	10000 4000 10000 4100
 Wire Wire Line
-	10100 4250 10000 4250
-Wire Wire Line
-	10000 4250 10000 4100
-Connection ~ 10000 4100
-Wire Wire Line
 	4850 3600 5000 3600
 Text GLabel 4850 3600 0    50   Input ~ 0
@@
 F 0 "U3" H 2950 6642 50  0000 C CNN
 F 1 "LM1117-3.3" H 2950 6551 50  0000 C CNN
-F 2 "RF_Module:HOPERF_RFM69HW" H 2950 6400 50  0001 C CNN
+F 2 "lm1117t-3.3_nopb:TO254P470X1028X1955-3P" H 2950 6400 50  0001 C CNN
 F 3 "http://www.ti.com/lit/ds/symlink/lm1117.pdf" H 2950 6400 50  0001 C CNN
 	1    2950 6400
@@
 F 0 "J7" H 742 6275 50  0000 C CNN
 F 1 "PWR_IN" H 742 6366 50  0000 C CNN
-F 2 "Connector:Banana_Jack_2Pin" H 850 6600 50  0001 C CNN
+F 2 "Connector_Wire:SolderWirePad_1x02_P3.81mm_Drill1mm" H 850 6600 50  0001 C CNN
 F 3 "~" H 850 6600 50  0001 C CNN
 	1    850  6600
@@
 F 0 "SW1" H 1500 2285 50  0000 C CNN
 F 1 "RESET" H 1500 2194 50  0000 C CNN
-F 2 "" H 1500 2200 50  0001 C CNN
+F 2 "button:FSM4JRT" H 1500 2200 50  0001 C CNN
 F 3 "~" H 1500 2200 50  0001 C CNN
 	1    1500 2000
@@
 F 0 "SW2" V 3704 1948 50  0000 L CNN
 F 1 "PROGRAM" V 3795 1948 50  0000 L CNN
-F 2 "" H 3750 2000 50  0001 C CNN
+F 2 "button:FSM4JRT" H 3750 2000 50  0001 C CNN
 F 3 "~" H 3750 2000 50  0001 C CNN
 	1    3750 1800
@@
 Text GLabel 9750 4350 0    50   Input ~ 0
 LAUNCH2_OUT
-Wire Wire Line
-	9750 4350 10100 4350
 $Comp
 L Device:C C6
@@
 F 0 "J5" H 4778 6876 50  0000 L CNN
 F 1 "I2C_PRESSURE" H 4778 6785 50  0000 L CNN
-F 2 "Connector_PinSocket_2.54mm:PinSocket_1x04_P2.54mm_Vertical" H 4750 6700 50  0001 C CNN
+F 2 "custom:PinSocket_1x04_P2.54mm_Vertical" H 4750 6700 50  0001 C CNN
 F 3 "" H 4750 6700 50  0001 C CNN
 	1    4750 6700
@@
 F 0 "J8" H 4778 7626 50  0000 L CNN
 F 1 "I2C_GYRO" H 4778 7535 50  0000 L CNN
-F 2 "Connector_PinSocket_2.54mm:PinSocket_1x04_P2.54mm_Vertical" H 4750 7450 50  0001 C CNN
+F 2 "custom:PinSocket_1x04_P2.54mm_Vertical" H 4750 7450 50  0001 C CNN
 F 3 "" H 4750 7450 50  0001 C CNN
 	1    4750 7450
@@
 F 0 "J9" H 6178 7626 50  0000 L CNN
 F 1 "I2C_RTC" H 6178 7535 50  0000 L CNN
-F 2 "Connector_PinSocket_2.54mm:PinSocket_1x04_P2.54mm_Vertical" H 6150 7450 50  0001 C CNN
+F 2 "custom:PinSocket_1x04_P2.54mm_Vertical" H 6150 7450 50  0001 C CNN
 F 3 "" H 6150 7450 50  0001 C CNN
 	1    6150 7450
@@
 Wire Wire Line
 	950  6050 1200 6050
+Wire Wire Line
+	10000 4100 10000 4350
+Wire Wire Line
+	10000 4350 10100 4350
+Connection ~ 10000 4100
+Wire Wire Line
+	10100 4250 9850 4250
+Wire Wire Line
+	9850 4250 9850 4350
+Wire Wire Line
+	9850 4350 9750 4350
 $EndSCHEMATC

Commit message: Use smaller components
Parts:
- removed J6: SD_Card, Connector_Card:SD_TE_2041021, symbol Connector:SD_Card
- added J6: Micro_SD_Card, Connector_Card:microSD_HC_Molex_104031-0811, symbol Connector:Micro_SD_Card
- added R8, R9: 4K7, Resistor_SMD:R_0805_2012Metric_Pad1.15x1.40mm_HandSolder, symbol Device:R
- C1, C4, C5, C6, C7, C8, C9: footprint Capacitor_THT:C_Disc_D4.7mm_W2.5mm_P5.00mm -> Capacitor_SMD:C_0805_2012Metric_Pad1.15x1.40mm_HandSolder
- R1, R2, R3, R4, R5, R6, R7: footprint Resistor_THT:R_Axial_DIN0207_L6.3mm_D2.5mm_P7.62mm_Horizontal -> Resistor_SMD:R_0805_2012Metric_Pad1.15x1.40mm_HandSolder
Connections:
- net +3V3: now also J6.4 (VDD), J6.6 (VSS), R8.2, R9.2
- net CLK: now also J6.5 (CLK)
- net CS0: now also J6.2 (DAT3/CD)
- net GND: now also J6.9 (SHIELD)
- net MISO: now also J6.7 (DAT0)
- net MOSI: now also J6.3 (CMD)
- net SCL: now also R9.1
- net SDA: now also R8.1
- no-connect marks 25 -> 23
Changed lines of the file:
@@
 Wire Wire Line
 	10000 4000 10000 4100
-Wire Wire Line
-	4850 3600 5000 3600
-Text GLabel 4850 3600 0    50   Input ~ 0
+Text GLabel 4950 3350 0    50   Input ~ 0
 MISO
-Wire Wire Line
-	4650 3100 5000 3100
-Text GLabel 4650 3100 0    50   Input ~ 0
-MOSI
-Wire Wire Line
-	4850 3000 5000 3000
-$Comp
-L power:+3V3 #PWR03
-U 1 1 5E79C103
-P 4750 3300
-F 0 "#PWR03" H 4750 3150 50  0001 C CNN
-F 1 "+3V3" H 4765 3473 50  0000 C CNN
-F 2 "" H 4750 3300 50  0001 C CNN
-F 3 "" H 4750 3300 50  0001 C CNN
-	1    4750 3300
-	1    0    0    -1
-$EndComp
-Wire Wire Line
-	4850 3400 5000 3400
-Text GLabel 4850 3400 0    50   Input ~ 0
-CLK
-Text GLabel 4850 3000 0    50   Input ~ 0
+Text GLabel 4950 2850 0    50   Input ~ 0
 CS0
-Wire Wire Line
-	7150 3500 7150 3550
-Wire Wire Line
-	6800 3500 7150 3500
-Connection ~ 7150 3500
-Wire Wire Line
-	7150 3400 7150 3500
-Wire Wire Line
-	6800 3400 7150 3400
-$Comp
-L power:GND #PWR07
-U 1 1 5E78B0CA
-P 7150 3550
-F 0 "#PWR07" H 7150 3300 50  0001 C CNN
-F 1 "GND" H 7155 3377 50  0000 C CNN
-F 2 "" H 7150 3550 50  0001 C CNN
-F 3 "" H 7150 3550 50  0001 C CNN
-	1    7150 3550
-	1    0    0    -1
-$EndComp
-Wire Wire Line
-	4750 3300 5000 3300
-Wire Wire Line
-	5000 3200 4900 3200
-Wire Wire Line
-	4900 3200 4900 3500
-Wire Wire Line
-	4900 3500 4900 3850
-Connection ~ 4900 3500
-Wire Wire Line
-	5000 3500 4900 3500
-$Comp
-L power:GND #PWR04
-U 1 1 5E77C249
-P 4900 3850
-F 0 "#PWR04" H 4900 3600 50  0001 C CNN
-F 1 "GND" H 4905 3677 50  0000 C CNN
-F 2 "" H 4900 3850 50  0001 C CNN
-F 3 "" H 4900 3850 50  0001 C CNN
-	1    4900 3850
-	1    0    0    -1
-$EndComp
-$Comp
-L Connector:SD_Card J6
-U 1 1 5E778F11
-P 5900 3300
-F 0 "J6" H 5900 3965 50  0000 C CNN
-F 1 "SD_Card" H 5900 3874 50  0000 C CNN
-F 2 "Connector_Card:SD_TE_2041021" H 5900 3300 50  0001 C CNN
-F 3 "http://portal.fciconnect.com/Comergent//fci/drawing/10067847.pdf" H 5900 3300 50  0001 C CNN
-	1    5900 3300
-	1    0    0    -1
-$EndComp
 Text GLabel 9650 1500 0    50   Input ~ 0
 LAUNCH1
@@
 F 0 "C4" H 6865 4846 50  0000 L CNN
 F 1 "100nF" H 6865 4755 50  0000 L CNN
-F 2 "Capacitor_THT:C_Disc_D4.7mm_W2.5mm_P5.00mm" H 6788 4650 50  0001 C CNN
+F 2 "Capacitor_SMD:C_0805_2012Metric_Pad1.15x1.40mm_HandSolder" H 6788 4650 50  0001 C CNN
 F 3 "~" H 6750 4800 50  0001 C CNN
 	1    6750 4800
@@
 F 0 "R3" V 9693 1500 50  0000 C CNN
 F 1 "10K" V 9784 1500 50  0000 C CNN
-F 2 "Resistor_THT:R_Axial_DIN0207_L6.3mm_D2.5mm_P7.62mm_Horizontal" V 9830 1500 50  0001 C CNN
+F 2 "Resistor_SMD:R_0805_2012Metric_Pad1.15x1.40mm_HandSolder" V 9830 1500 50  0001 C CNN
 F 3 "~" H 9900 1500 50  0001 C CNN
 	1    9900 1500
@@
 F 0 "R4" H 10520 1046 50  0000 L CNN
 F 1 "10K" H 10520 955 50  0000 L CNN
-F 2 "Resistor_THT:R_Axial_DIN0207_L6.3mm_D2.5mm_P7.62mm_Horizontal" V 10380 1000 50  0001 C CNN
+F 2 "Resistor_SMD:R_0805_2012Metric_Pad1.15x1.40mm_HandSolder" V 10380 1000 50  0001 C CNN
 F 3 "~" H 10450 1000 50  0001 C CNN
 	1    10450 1000
@@
 F 0 "R2" V 9693 950 50  0000 C CNN
 F 1 "100R" V 9784 950 50  0000 C CNN
-F 2 "Resistor_THT:R_Axial_DIN0207_L6.3mm_D2.5mm_P7.62mm_Horizontal" V 9830 950 50  0001 C CNN
+F 2 "Resistor_SMD:R_0805_2012Metric_Pad1.15x1.40mm_HandSolder" V 9830 950 50  0001 C CNN
 F 3 "~" H 9900 950 50  0001 C CNN
 	1    9900 950
@@
 F 0 "C1" H 1965 3196 50  0000 L CNN
 F 1 "100nF" H 1965 3105 50  0000 L CNN
-F 2 "Capacitor_THT:C_Disc_D4.7mm_W2.5mm_P5.00mm" H 1888 3000 50  0001 C CNN
+F 2 "Capacitor_SMD:C_0805_2012Metric_Pad1.15x1.40mm_HandSolder" H 1888 3000 50  0001 C CNN
 F 3 "~" H 1850 3150 50  0001 C CNN
 	1    1850 3150
@@
 F 0 "R1" H 2170 1796 50  0000 L CNN
 F 1 "10KR" H 2170 1705 50  0000 L CNN
-F 2 "Resistor_THT:R_Axial_DIN0207_L6.3mm_D2.5mm_P7.62mm_Horizontal" V 2030 1750 50  0001 C CNN
+F 2 "Resistor_SMD:R_0805_2012Metric_Pad1.15x1.40mm_HandSolder" V 2030 1750 50  0001 C CNN
 F 3 "~" H 2100 1750 50  0001 C CNN
 	1    2100 1750
@@
 F 0 "R6" V 9693 3100 50  0000 C CNN
 F 1 "10K" V 9784 3100 50  0000 C CNN
-F 2 "Resistor_THT:R_Axial_DIN0207_L6.3mm_D2.5mm_P7.62mm_Horizontal" V 9830 3100 50  0001 C CNN
+F 2 "Resistor_SMD:R_0805_2012Metric_Pad1.15x1.40mm_HandSolder" V 9830 3100 50  0001 C CNN
 F 3 "~" H 9900 3100 50  0001 C CNN
 	1    9900 3100
@@
 F 0 "R7" H 10520 2646 50  0000 L CNN
 F 1 "10K" H 10520 2555 50  0000 L CNN
-F 2 "Resistor_THT:R_Axial_DIN0207_L6.3mm_D2.5mm_P7.62mm_Horizontal" V 10380 2600 50  0001 C CNN
+F 2 "Resistor_SMD:R_0805_2012Metric_Pad1.15x1.40mm_HandSolder" V 10380 2600 50  0001 C CNN
 F 3 "~" H 10450 2600 50  0001 C CNN
 	1    10450 2600
@@
 F 0 "R5" V 9693 2550 50  0000 C CNN
 F 1 "100R" V 9784 2550 50  0000 C CNN
-F 2 "Resistor_THT:R_Axial_DIN0207_L6.3mm_D2.5mm_P7.62mm_Horizontal" V 9830 2550 50  0001 C CNN
+F 2 "Resistor_SMD:R_0805_2012Metric_Pad1.15x1.40mm_HandSolder" V 9830 2550 50  0001 C CNN
 F 3 "~" H 9900 2550 50  0001 C CNN
 	1    9900 2550
@@
 F 0 "C6" H 4765 1196 50  0000 L CNN
 F 1 "100nF" H 4765 1105 50  0000 L CNN
-F 2 "Capacitor_THT:C_Disc_D4.7mm_W2.5mm_P5.00mm" H 4688 1000 50  0001 C CNN
+F 2 "Capacitor_SMD:C_0805_2012Metric_Pad1.15x1.40mm_HandSolder" H 4688 1000 50  0001 C CNN
 F 3 "~" H 4650 1150 50  0001 C CNN
 	1    4650 1150
@@
 F 0 "C7" H 4765 2046 50  0000 L CNN
 F 1 "100nF" H 4765 1955 50  0000 L CNN
-F 2 "Capacitor_THT:C_Disc_D4.7mm_W2.5mm_P5.00mm" H 4688 1850 50  0001 C CNN
+F 2 "Capacitor_SMD:C_0805_2012Metric_Pad1.15x1.40mm_HandSolder" H 4688 1850 50  0001 C CNN
 F 3 "~" H 4650 2000 50  0001 C CNN
 	1    4650 2000
@@
 SDA
 Wire Wire Line
-	3550 4200 3650 4200
-Wire Wire Line
-	3550 4300 3650 4300
+	3550 4200 3600 4200
+Wire Wire Line
+	3550 4300 3600 4300
 Text GLabel 4200 6600 0    50   Input ~ 0
 SCL
@@
 F 0 "C5" H 4165 6396 50  0000 L CNN
 F 1 "100nF" H 4165 6305 50  0000 L CNN
-F 2 "Capacitor_THT:C_Disc_D4.7mm_W2.5mm_P5.00mm" H 4088 6200 50  0001 C CNN
+F 2 "Capacitor_SMD:C_0805_2012Metric_Pad1.15x1.40mm_HandSolder" H 4088 6200 50  0001 C CNN
 F 3 "~" H 4050 6350 50  0001 C CNN
 	1    4050 6350
@@
 F 0 "C8" H 4165 7146 50  0000 L CNN
 F 1 "100nF" H 4165 7055 50  0000 L CNN
-F 2 "Capacitor_THT:C_Disc_D4.7mm_W2.5mm_P5.00mm" H 4088 6950 50  0001 C CNN
+F 2 "Capacitor_SMD:C_0805_2012Metric_Pad1.15x1.40mm_HandSolder" H 4088 6950 50  0001 C CNN
 F 3 "~" H 4050 7100 50  0001 C CNN
 	1    4050 7100
@@
 F 0 "C9" H 5565 7146 50  0000 L CNN
 F 1 "100nF" H 5565 7055 50  0000 L CNN
-F 2 "Capacitor_THT:C_Disc_D4.7mm_W2.5mm_P5.00mm" H 5488 6950 50  0001 C CNN
+F 2 "Capacitor_SMD:C_0805_2012Metric_Pad1.15x1.40mm_HandSolder" H 5488 6950 50  0001 C CNN
 F 3 "~" H 5450 7100 50  0001 C CNN
 	1    5450 7100
@@
 Wire Wire Line
 	6400 4500 7100 4500
-NoConn ~ 6800 3200
-NoConn ~ 6800 3100
-NoConn ~ 5000 3700
-NoConn ~ 5000 2900
 NoConn ~ 6400 5100
 NoConn ~ 6400 5000
@@
 Wire Wire Line
 	9850 4350 9750 4350
+$Comp
+L power:+3V3 #PWR023
+U 1 1 5EAB72B7
+P 3850 4650
+F 0 "#PWR023" H 3850 4500 50  0001 C CNN
+F 1 "+3V3" H 3865 4823 50  0000 C CNN
+F 2 "" H 3850 4650 50  0001 C CNN
+F 3 "" H 3850 4650 50  0001 C CNN
+	1    3850 4650
+	0    1    1    0
+$EndComp
+$Comp
+L Device:R R9
+U 1 1 5EAB7AB7
+P 4150 4350
+F 0 "R9" H 4220 4396 50  0000 L CNN
+F 1 "4K7" H 4220 4305 50  0000 L CNN
+F 2 "Resistor_SMD:R_0805_2012Metric_Pad1.15x1.40mm_HandSolder" V 4080 4350 50  0001 C CNN
+F 3 "~" H 4150 4350 50  0001 C CNN
+	1    4150 4350
+	1    0    0    -1
+$EndComp
+$Comp
+L Device:R R8
+U 1 1 5EAB86BE
+P 3600 4550
+F 0 "R8" H 3670 4596 50  0000 L CNN
+F 1 "4K7" H 3670 4505 50  0000 L CNN
+F 2 "Resistor_SMD:R_0805_2012Metric_Pad1.15x1.40mm_HandSolder" V 3530 4550 50  0001 C CNN
+F 3 "~" H 3600 4550 50  0001 C CNN
+	1    3600 4550
+	1    0    0    -1
+$EndComp
+Wire Wire Line
+	3600 4300 3600 4400
+Connection ~ 3600 4300
+Wire Wire Line
+	3600 4300 3650 4300
+Wire Wire Line
+	3600 4700 3800 4700
+Wire Wire Line
+	3850 4700 3850 4650
+Wire Wire Line
+	3600 4200 3600 4100
+Wire Wire Line
+	3600 4100 4150 4100
+Wire Wire Line
+	4150 4100 4150 4200
+Connection ~ 3600 4200
+Wire Wire Line
+	3600 4200 3650 4200
+Wire Wire Line
+	4150 4500 3800 4500
+Wire Wire Line
+	3800 4500 3800 4700
+Connection ~ 3800 4700
+Wire Wire Line
+	3800 4700 3850 4700
+$Comp
+L Connector:Micro_SD_Card J6
+U 1 1 5EB45DB9
+P 5950 3050
+F 0 "J6" H 5900 3767 50  0000 C CNN
+F 1 "Micro_SD_Card" H 5900 3676 50  0000 C CNN
+F 2 "Connector_Card:microSD_HC_Molex_104031-0811" H 7100 3350 50  0001 C CNN
+F 3 "http://katalog.we-online.de/em/datasheet/693072010801.pdf" H 5950 3050 50  0001 C CNN
+	1    5950 3050
+	1    0    0    -1
+$EndComp
+Text GLabel 4950 2950 0    50   Input ~ 0
+MOSI
+Text GLabel 4950 3150 0    50   Input ~ 0
+CLK
+$Comp
+L power:+3V3 #PWR03
+U 1 1 5E79C103
+P 4750 3050
+F 0 "#PWR03" H 4750 2900 50  0001 C CNN
+F 1 "+3V3" H 4765 3223 50  0000 C CNN
+F 2 "" H 4750 3050 50  0001 C CNN
+F 3 "" H 4750 3050 50  0001 C CNN
+	1    4750 3050
+	0    -1   -1   0
+$EndComp
+Wire Wire Line
+	5050 3250 4700 3250
+Wire Wire Line
+	4700 3250 4700 3050
+Wire Wire Line
+	4700 3050 4750 3050
+Wire Wire Line
+	4750 3050 5050 3050
+Connection ~ 4750 3050
+Wire Wire Line
+	4950 2950 5050 2950
+Wire Wire Line
+	4950 2850 5050 2850
+NoConn ~ 5050 2750
+NoConn ~ 5050 3450
+Wire Wire Line
+	4950 3350 5050 3350
+Wire Wire Line
+	4950 3150 5050 3150
+$Comp
+L power:GND #PWR04
+U 1 1 5EBDAA45
+P 6750 3750
+F 0 "#PWR04" H 6750 3500 50  0001 C CNN
+F 1 "GND" H 6755 3577 50  0000 C CNN
+F 2 "" H 6750 3750 50  0001 C CNN
+F 3 "" H 6750 3750 50  0001 C CNN
+	1    6750 3750
+	1    0    0    -1
+$EndComp
+Wire Wire Line
+	6750 3650 6750 3750
 $EndSCHEMATC

Commit message: Edited the PCB design
Parts:
- J5, J8, J9: symbol ConnectorCustom:I2C_CONN -> RocketTracker-rescue:I2C_CONN-ConnectorCustom
- Q1, Q3: symbol dk_Transistors-FETs-MOSFETs-Single:FQP27P06 -> RocketTracker-rescue:FQP27P06-dk_Transistors-FETs-MOSFETs-Single
Changed lines of the file:
@@
 $EndComp
 $Comp
-L dk_Transistors-FETs-MOSFETs-Single:FQP27P06 Q3
+L RocketTracker-rescue:FQP27P06-dk_Transistors-FETs-MOSFETs-Single Q3
 U 1 1 5EA3C4BC
 P 9000 2650
@@
 	4650 2150 5450 2150
 $Comp
-L ConnectorCustom:I2C_CONN J5
+L RocketTracker-rescue:I2C_CONN-ConnectorCustom J5
 U 1 1 5EB19821
 P 4750 6700
@@
 	4500 7150 4550 7150
 $Comp
-L ConnectorCustom:I2C_CONN J8
+L RocketTracker-rescue:I2C_CONN-ConnectorCustom J8
 U 1 1 5EB1C8B6
 P 4750 7450
@@
 	5900 7150 5950 7150
 $Comp
-L ConnectorCustom:I2C_CONN J9
+L RocketTracker-rescue:I2C_CONN-ConnectorCustom J9
 U 1 1 5EB28A43
 P 6150 7450
@@
 NoConn ~ 2350 2300
 $Comp
-L dk_Transistors-FETs-MOSFETs-Single:FQP27P06 Q1
+L RocketTracker-rescue:FQP27P06-dk_Transistors-FETs-MOSFETs-Single Q1
 U 1 1 5E9EA243
 P 9000 1050
